File: HW/V0.0/Power_Peripherals.kicad_sch (KiCad schematic)
At the start: 54 parts, among them Q10 TVS_2CH, Q3 <name>, Q4 <name>, Q5 <name>, Q6 <name>, Q7 <name>, U1 3.3V/300mA, U5 28V/3A Bck

Commit message: PIC16-DevKit-SCH-877 schematic update 2
Parts:
- removed Q5, Q7: <name>, symbol Triet_KiCAD_Sym:PNP
- removed R14, R15: 10k, symbol Triet_KiCAD_Sym:RES
Connections:
- net +5V: no longer C24.1, C27.1, C28.1, L1.2, R19.1, R36.2
- net USB+ renamed USB_P
- net USB- renamed USB_N
- new net: C24.1, C27.1, C28.1, L1.2, R19.1, R36.2
