File: HW/V0.0/Target_MCU.kicad_sch (KiCad schematic)
At the start: 36 parts, among them J3 EXP PORT, J5 QWIIC, Q6 SI2302, Q7 SI2302, U10 20MHz, U4 PIC16F877A

Commit message: PIC16-DevKit-PCB-877 layout update 1
Connections:
- net GPIO: now also U4.27 (RE2/~{CS}/AN7)
- net SCLK: now also U4.15 (RB5)
- net SDI: now also U4.14 (RB4)
- net ~{CS}: now also U4.26 (RE1/~{WR}/AN6)
Changed lines of the file:
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@@
 	(hierarchical_label "~{CS}"
 		(shape output)
-		(at 60.96 90.17 180)
+		(at 62.23 90.17 180)
 		(fields_autoplaced yes)
 		(effects
@@
 	(hierarchical_label "GPIO"
 		(shape output)
-		(at 60.325 93.98 180)
+		(at 62.23 93.98 180)
 		(fields_autoplaced yes)
 		(effects
@@
 	(hierarchical_label "SCLK"
 		(shape output)
-		(at 115.57 78.74 0)
+		(at 113.03 78.74 0)
 		(fields_autoplaced yes)
 		(effects
@@
 	(hierarchical_label "SDI"
 		(shape input)
-		(at 115.57 74.93 0)
+		(at 113.03 74.93 0)
 		(fields_autoplaced yes)
 		(effects
@@
 		)
 		(instances
-			(project ""
+			(project "PIC16DevKit"
 				(path "/17281b91-3f9a-4e36-96b2-66002b412b3a/dceb7a93-1172-4461-96bc-c129bdd90128"
 					(reference "J5")
