File: HW/Design/V0.0/PIC16DevKit.kicad_pcb (KiCad board)
At the start: 4 copper layers, 68.8 x 54 mm, 100 parts, among them J1 9V-12V, J2 USB C, J3 EXP PORT, J4 SIL04, J5 QWIIC, Q1 SI2301, Q3 SI2301, Q4 2N3906, Q5 SI2302, Q6 SI2302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

Commit message: PIC16-DevKit-PCB-877 layout update 3
Routing:
- net GND: track 28.8 -> 44.8 mm, vias 16 -> 207

Commit message: PIC16-DevKit-PCB-877 layout update 4
Parts:
- C1: value 470uF -> 220uF; footprint SAMPI:CAP_ELEC-8.3x8.3-DIA8.0 -> SAMPI:CAP_ELEC-6.6x6.6-DIA6.3
- moved G*** 0.15 mm to (119.5, 54.2)
- turned Q3 to 0 degrees
Connections:
- R19 pad 1: +5V -> +VDDTG
- R27 pad 1: +5V -> +VDDTG
Routing:
- net VBUS: track 32.6 -> 56.5 mm, vias 3 -> 6
- net +VDDTG: track 182.1 -> 202.3 mm, vias 6 -> 7
- net +5V: track 144.3 -> 133.4 mm
- net GND: track 44.8 -> 38.2 mm, vias 207 -> 227
- net Net-(U2-SW): track 16.6 -> 11.7 mm
- net Net-(Q3-G): track 9.79 -> 6.07 mm
- net /PROGRAMMER/RXD0: track 23.2 -> 21.5 mm
- net /PROGRAMMER/SDA: track 87.7 -> 86.2 mm
- net +3.3V: track 76.0 -> 77.0 mm, vias 3 -> 4
- net Net-(U3-SW): track 8.46 -> 9.48 mm
- net /PROGRAMMER/TXD0: track 23.8 -> 23.0 mm
- added copper zone on F.Cu, net VBUS
- removed copper zone on B.Cu, net +5V
- removed copper zone on In1.Cu, net +5V
Other:
- board text added: "PIC16F877A"
