File: HW/Design/V0.0/PIC16DevKit.kicad_pcb (KiCad board)
At the start: 4 copper layers, 68.8 x 54 mm, 100 parts, among them J1 9V-12V, J2 USB C, J3 EXP PORT, J4 SIL04, J5 QWIIC, Q1 SI2301, Q3 SI2301, Q4 2N3906, Q5 SI2302, Q6 SI2302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

Commit message: PIC16-DevKit-PCB-877 PCB V0.0
Parts:
- added G***: LOGO, LOGO, F.Cu at (111.5, 82.8)
- added G***: LOGO, LOGO, B.Cu at (125.1, 54.0)
- added G***: LOGO, LOGO, B.Cu at (103.1, 70.0)
- added TP1: PGC/B6, SAMPI:TP1MM, B.Cu at (77.0, 64.9)
- added TP2: PGD/B7, SAMPI:TP1MM, B.Cu at (77.6, 62.6)
- BT1: value MODE -> FNC
- moved G*** 0.25 mm to (119.5, 54.4)
Connections:
- net /PROGRAMMER/~{BT_MODE} renamed /PROGRAMMER/~{BT_FNC}
- MD1 pad 21: /TARGET MCU/INT0 -> /TARGET MCU/INT1
- MD1 pad 22: /TARGET MCU/INT1 -> /TARGET MCU/INT0
Routing:
- net /TARGET MCU/INT1: track 39.2 -> 34.6 mm
- net /TARGET MCU/INT0: track 34.1 -> 36.2 mm
- net /PROGRAMMER/TG_PGD: track 37.5 -> 38.2 mm
- net GND: vias 227 -> 221
Other:
- board text added: "A0/AN0"
- board text added: "A1/AN1"
- board text added: "A2/AN2"
- board text added: "A3/AN3"
- board text added: "A4"
- board text added: "A5/AN4"
- board text added: "B0"
- board text added: "B1"
- board text added: "B2"
- board text added: "B3"
- board text added: "B4"
- board text added: "B5"
- board text added: "C0"
- board text added: "C1"
- board text added: "C2"
- board text added: "C3"
- board text added: "C4"
- board text added: "C5"
- board text added: "C6"
- board text added: "C7"
- board text added: "E0/AN5"
- board text added: "E1/AN6"
- board text added: "E2/AN7"
- board text added: "GPIO"
- board text added: "PCB V0.0"
- board text added: "PIC16F877A DEV KIT V0"
- board text added: "SDO"
- board text added: "TXD"
- board text removed: "GPIO0"
- board text removed: "PIC16F877A"
- board text removed: "RXD1"
- board text removed: "SD0"
- board text removed: "TXD1"

Commit message: PIC16-DevKit-PCB-877 layout update 5
Routing:
- net +5V: track 133.4 -> 142.2 mm
- net +VDDTG: track 202.3 -> 209.2 mm
- net +3.3V: track 77.0 -> 74.6 mm
- net GND: track 38.2 -> 40.0 mm, vias 221 -> 224
