File: HW/Design/V0.0/POWER.kicad_sch (KiCad schematic)
At the start: 44 parts, among them J1 9V-12V, J2 USB C, Q1 SI2301, Q3 SI2301, Q4 2N3906, U1 LDO 3.3V/300mA, U2 MT1470, U3 MT3608

Commit message: PIC16-DevKit-PCB-877 layout update 4
Parts:
- C1: value 470uF -> 220uF; footprint SAMPI:CAP_ELEC-8.3x8.3-DIA8.0 -> SAMPI:CAP_ELEC-6.6x6.6-DIA6.3; MNP EXV477M016A9MAA -> EEV227M016S9HAA
Changed lines of the file:
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@@
 			)
 		)
-		(property "Value" "470uF"
+		(property "Value" "220uF"
 			(at 65.405 35.56 90)
 			(effects
@@
 			)
 		)
-		(property "Footprint" "SAMPI:CAP_ELEC-8.3x8.3-DIA8.0"
+		(property "Footprint" "SAMPI:CAP_ELEC-6.6x6.6-DIA6.3"
 			(at 64.77 33.02 0)
 			(effects
@@
 			)
 		)
-		(property "Description" "CAP ALUM 470UF 20% 16V SMD"
+		(property "Description" "CAP ALUM 220UF 20% 16V SMD"
 			(at 64.77 33.02 0)
 			(effects
@@
 			)
 		)
-		(property "MNP" "EXV477M016A9MAA"
+		(property "MNP" "EEV227M016S9HAA"
 			(at 64.77 33.02 0)
 			(effects

Commit message: PIC16-DevKit-PCB-877 PCB V0.0
Other:
- company: (none) -> SAMPI DEVELOPMENT KITS
- title: (none) -> PIC16F877A DEV KIT
Changed lines of the file:
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@@
 	(generator_version "8.0")
 	(paper "A4")
+	(title_block
+		(title "PIC16F877A DEV KIT")
+		(date "2025-01-01")
+		(rev "0.0")
+		(company "SAMPI DEVELOPMENT KITS")
+		(comment 1 "P/N: SAMM-16F877A")
+	)
 	(junction
 		(at 50.8 82.55)

Commit message: PIC16-DevKit-PCB-877 V0.1 - QWIIC ESD protection, disable VPP, detect VBUS, measure VPP, VDDTG
Parts:
- added C40, C41: 100nF, SAMPI:CAP0603, symbol Triet_KiCAD_Sym:CAP_CER
- added R31: 100K, SAMPI:RES0603, symbol Triet_KiCAD_Sym:RES
- added R34: 47K, 1%, SAMPI:RES0603, symbol Triet_KiCAD_Sym:RES
- added R35: 5.1K, 1%, SAMPI:RES0603, symbol Triet_KiCAD_Sym:RES
- added R36: 10K, 1%, SAMPI:RES0603, symbol Triet_KiCAD_Sym:RES
- R32: value 10K, 1% -> 5.1K, 1%; MNP RC0603FR-0710KL -> RC0603FR-075K1L
- R33: value 10K, 1% -> 47K, 1%; MNP RC0603FR-0710KL -> RC0603FR-0747KL
Connections:
- net +VDDTG: now also R34.1
- net GND: now also C40.2, C41.2, R31.2, R35.2
- net VPP_EN: now also R31.1
- net at C12.2, R10.1, R5.2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: now also R36.1
- net VBUS_SEN renamed VBUS_DIV
- new net VDDTG_DIV: C40.1, R34.2, R35.1
- new net VPP_DIV: C41.1, R36.2
