File: HW/Design/V0.1/Target_MCU.kicad_sch (KiCad schematic)
At the start: 36 parts, among them J3 EXP PORT, J5 QWIIC, Q6 SI2302, Q7 SI2302, U10 20MHz, U4 PIC16F877A

Commit message: Update diagram
Parts:
- added D5: TVS 5V, SAMPI:SOT143B_NEXT, symbol SAMPI:TVS_3CH
Connections:
- net +3.3V: now also D5.4 (CH3)
- net GND: now also D5.1 (GND)
- net at J5.4 (SCL), Q6.2 (S), R28.2: now also D5.2 (CH1)
- net at J5.3 (SDA), Q7.2 (S), R30.2: now also D5.3 (CH2)
Other:
- moved on the sheet: J5, Q6, Q7, R21, R22, R28, R30
