File: HW/Design/V0.1/POWER.kicad_sch (KiCad schematic)
At the start: 44 parts, among them J1 9V-12V, J2 USB C, Q1 SI2301, Q3 SI2301, Q4 2N3906, U1 LDO 3.3V/300mA, U2 MT1470, U3 MT3608

Commit message: Update diagram
Parts:
- added C41: 100nF, SAMPI:CAP0603, symbol Triet_KiCAD_Sym:CAP_CER
- added R31: 100K, SAMPI:RES0603, symbol Triet_KiCAD_Sym:RES
- added R32, R35: 5.1K, 1%, SAMPI:RES0603, symbol Triet_KiCAD_Sym:RES
- added R34: 47K, 1%, SAMPI:RES0603, symbol Triet_KiCAD_Sym:RES
- added R36: 10K, 1%, SAMPI:RES0603, symbol Triet_KiCAD_Sym:RES
- C40: value 1uF -> 100nF
- R33: value DNM -> 47K, 1%; MNP RC0603FR-0710KL -> RC0603FR-0747KL; now fitted; now in the parts list
Connections:
- net +VDDTG: now also R34.1
- net GND: now also C41.2, R31.2, R32.2, R35.2
- net VPP_EN: now also R31.1
- net at C12.2, R10.1, R5.2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: now also R36.1
- net VBUS_SEN renamed VBUS_DIV
- net VBUS_DIV: now also R32.1; no longer C40.1
- new net VDDTG_DIV: C40.1, R34.2, R35.1
- new net VPP_DIV: C41.1, R36.2
Other:
- note removed: "Place close to MCU pin"

Commit message: AVR64DU28 bootloader update 2
Parts:
- removed C1: 220uF, SAMPI:CAP_ELEC-6.6x6.6-DIA6.3, symbol SAMPI:ELECCAP
- removed C10, C11, C13, C7, C8, C9: 10uF, SAMPI:CAP0603, symbol Triet_KiCAD_Sym:CAP_CER
- removed C12: 22pF, SAMPI:CAP0603, symbol Triet_KiCAD_Sym:CAP_CER
- removed C14, C38, C39, C4, C40, C41, C5, C6: 100nF, SAMPI:CAP0603, symbol Triet_KiCAD_Sym:CAP_CER
- removed C2: 220uF, SAMPI:CAP1411, symbol SAMPI:ELECCAP
- removed C3: 10uF/16V, SAMPI:CAP1206, symbol Triet_KiCAD_Sym:CAP_CER
- removed D1: 5V1, SAMPI:SOD80C-LL34, symbol SAMPI:DIODE-ZEN
- removed D2, D4: 200mA/0.2VF, SAMPI:SOD-123FL, symbol SAMPI:BAT42
- removed D3: TVS 5V, SAMPI:SOT143B_NEXT, symbol SAMPI:TVS_3CH
- removed F1: 1A, SAMPI:FUSE1812, symbol Triet_KiCAD_Sym:Fuse
- removed F2: 500mA, SAMPI:FUSE1812, symbol Triet_KiCAD_Sym:Fuse
- removed J1: 9V-12V, SAMPI:PJ-002AH-SMT, symbol Triet_KiCAD_Sym:PJ-002AH-SMT-TR
- removed J2: USB C, SAMPI:USB4105, symbol SAMPI:USB4105
- removed L1: 10uH/1.4A, SAMPI:IND5852, symbol SAMPI:IND
- removed L2: 10uH/100mA, SAMPI:IND0805, symbol SAMPI:IND
- removed Q1, Q3: SI2301, SAMPI:SOT23, symbol Triet_KiCAD_Sym:Mosfet-Pch
- removed Q4: 2N3906, SAMPI:SOT23, symbol SAMPI:BJT-PNP
- removed R1: 52.3K, 1%, SAMPI:RES0603, symbol Triet_KiCAD_Sym:RES
- removed R10, R2, R36: 10K, 1%, SAMPI:RES0603, symbol Triet_KiCAD_Sym:RES
- removed R3, R31, R8, R9: 100K, SAMPI:RES0603, symbol Triet_KiCAD_Sym:RES
- removed R32, R35, R6, R7: 5.1K, 1%, SAMPI:RES0603, symbol Triet_KiCAD_Sym:RES
- removed R33, R34: 47K, 1%, SAMPI:RES0603, symbol Triet_KiCAD_Sym:RES
- removed R4: 10K, SAMPI:RES0603, symbol Triet_KiCAD_Sym:RES
- removed R5: 191K, 1%, SAMPI:RES0603, symbol Triet_KiCAD_Sym:RES
- removed U1: LDO 3.3V/300mA, SAMPI:SOT-23-5_MCHP, symbol SAMPI:MIC5504_RT9193
- removed U2: MT1470, SAMPI:SOT-23-6_MCHP, symbol SAMPI:MT1470
- removed U3: MT3608, SAMPI:SOT-23-6_MCHP, symbol SAMPI:MT3608
Connections:
- no-connect marks 2 -> 0
Other:
- note removed: "Vo=0.6*(1+Rt/Rb) =0.6*(1+191/10) =12.06V"
- company: SAMPI DEVELOPMENT KITS -> (none)
- title: PIC16F877A DEV KIT -> USB TO DUAL SERIAL PORT & I2C
