File: HW/Design/V0.1/Programmer.kicad_sch (KiCad schematic)
At the start: 21 parts, among them J4 SIL04, Q5 SI2302, U5 AVRxxDU28

Commit message: Update diagram
Parts:
- added C23: 470nF, SAMPI:CAP0603, symbol Triet_KiCAD_Sym:CAP_CER
Connections:
- net GND: now also C23.2
- net VPP_SEN: now reaches U5.10 (PD0/ACINN/AIN7)
- net VDDTG_SEN: now reaches U5.11 (PD1/AIN8)
- net VBUS_DET: now reaches U5.9 (PC3/ACINP/AIN6)
- net USB_VBUS: no longer names the net of U5.6 (VUSB)
- net USB_VBUS: now also C23.1
- no-connect marks 5 -> 2

Commit message: AVR64DU28 bootloader update 2
Parts:
- removed C32, C37: 100nF, SAMPI:CAP0603, symbol Triet_KiCAD_Sym:CAP_CER
- removed J4: SIL04, SAMPI:HD-1x4x1.27MM-TH, symbol SAMPI:SIL04-1
- removed Q5: SI2302, SAMPI:SOT23, symbol SAMPI:FET_N-CH
- removed R19, R27: 5.1K, 1%, SAMPI:RES0603, symbol Triet_KiCAD_Sym:RES
- removed R26: 10K, SAMPI:RES0603, symbol Triet_KiCAD_Sym:RES
- removed R29: 330R, SAMPI:RES0603, symbol Triet_KiCAD_Sym:RES
- removed TP1: PGC/B6, SAMPI:TP1MM, symbol SAMPI:TESTPOINT
- removed TP2: PGD/B7, SAMPI:TP1MM, symbol SAMPI:TESTPOINT
- added C1: 100nF, SAMPI:CAP0603, symbol Triet_KiCAD_Sym:CAP_CER
- added D1, D2, D3, D4, D5, D7: 5.1V, Liem:SOD-323_12, symbol SAMPI:TVS
- added D6: TVS 5V, SAMPI:SOT143B_NEXT, symbol SAMPI:TVS_3CH
- added F1: 500mA, SAMPI:FUSE1812, symbol Triet_KiCAD_Sym:Fuse
- added J1: USB C, SAMPI:USB4105, symbol SAMPI:USB4105
- added J2: TERMINAL, symbol SAMPI:SIL08
- added J3: ICSP, symbol SAMPI:SIL08
- added MD1: PICKIT5, symbol SAMPI:SNAP-PG164100
- added R1, R3, R6: 5.1K, 1%, SAMPI:RES0603, symbol Triet_KiCAD_Sym:RES
- added R2, R4: 2.2K, SAMPI:RES0603, symbol Triet_KiCAD_Sym:RES
- added R5: 47K, 1%, SAMPI:RES0603, symbol Triet_KiCAD_Sym:RES
- renumbered C22 to C2, C25 to C3, C23 to C4, C26 to C5, C27 to C6, D6 to D8, D7 to D9, R24 to R7, R25 to R8, R23 to R9, U5 to U1
Connections:
- net +5V: now also D6.4 (CH3), F1.2, J2.2, J3.2, R2.1, R4.1, R5.1
- net GND: now also C1.2, D1.2, D2.2, D3.2, D4.2, D5.2, D6.1 (GND), D7.2, J1.A1B12 (GND), J1.B1A12 (GND), J1.S1, J1.S2, J1.S3, J1.S4, J2.1, J3.3, R1.2, R3.2, R6.2
- net RXD0: now also D3.1, J2.6
- net RXD1: now also D1.1, J2.8
- net SCL: now also D5.1, J2.4, R2.2
- net SDA: now also D7.1, J2.3, R4.2
- net TXD0: now also D4.1, J2.5
- net TXD1: now also D2.1, J2.7
- net USB_N: now also D6.3 (CH2), J1.A7 (DN1), J1.B7 (DN2)
- net USB_P: now also D6.2 (CH1), J1.A6 (DP1), J1.B6 (DP2)
- net VBUS_DET: now also C1.1, R5.2, R6.1
- net PG_UPDI: no longer names the net of U1.23 (PF7/UPDI)
- net PG_UPDI: now also J3.4
- net TG_MCLR: no longer names the net of U1.13 (PD3/ACINN/AIN10)
- net TG_PGC: no longer names the net of U1.26 (PA0/TX0/ASDA/XTALHF1)
- net TG_PGD: no longer names the net of U1.27 (PA1/RX0/ASCL/XTALHF2)
- net VDDTG_SEN: no longer names the net of U1.11 (PD1/AIN8)
- net VPP_EN: no longer names the net of U1.21 (PF1/ANI16/XTAL32K2)
- net VPP_SEN: no longer names the net of U1.10 (PD0/ACINN/AIN7)
- net ~{PG_RESET}: no longer names the net of U1.22 (PF6/~{RESET})
- net ~{PG_RESET}: now also J3.1
- net ~{VTG_EN}: no longer names the net of U1.20 (PF0/AIN15/XTAL32K1)
- new net: J1.B5 (CC2), R1.1
- new net: J1.A5 (CC1), R3.1
- new net: F1.1, J1.A4B9 (VBUS), J1.B4A9 (VBUS)
- no-connect marks 2 -> 15
Other:
- company: SAMPI DEVELOPMENT KITS -> (none)
- title: PIC16F877A DEV KIT -> USB TO DUAL SERIAL PORT & I2C
- moved on the sheet: BT1, C2, D8, D9, R7, R8, R9
