File: HW/Design/V1.0/Target_MCU.kicad_sch (KiCad schematic)
At the start: 36 parts, among them J3 EXP PORT, J5 QWIIC, Q6 SI2302, Q7 SI2302, U10 20MHz, U4 PIC16F877A

Commit message: PCB V2: change programmer MCU
Parts:
- removed C19, C21: 10uF, SAMPI:CAP0603, symbol Triet_KiCAD_Sym:CAP_CER
- removed R12, R13, R14, R15, R16, R17, R20: 330R, SAMPI:RES0603, symbol Triet_KiCAD_Sym:RES
- removed R21, R28, R30: 5.1K, 1%, SAMPI:RES0603, symbol Triet_KiCAD_Sym:RES
- added C14, C22: 100nF, SAMPI:CAP0603, symbol SAMPI:CERCAP
- added C21: 10uF, SAMPI:CAP0603, symbol SAMPI:CERCAP
- added R12, R13, R14, R15, R16, R17, R9: 1K, SAMPI:RES0603, symbol SAMPI:RES
- added R19, R20, R21, R23, R27: 5.1K, SAMPI:RES0603, symbol SAMPI:RES
- added R31, R32, R35: 330R, SAMPI:RES0603, symbol SAMPI:RES
- added R33: 10K, SAMPI:RES0603, symbol SAMPI:RES
- added R34: 10K, SAMPI:CDS-5MM, symbol SAMPI:CDS
- added U6: (no value), SAMPI:SOT23, symbol SAMPI:MCP9700-SOT23
- BT2: footprint Liem:SW6x6-G -> SAMPI:SW6x6-G
- C15, C16, C17, C18, C20: symbol Triet_KiCAD_Sym:CAP_CER -> SAMPI:CERCAP
- R11: value 330R -> 1K; symbol Triet_KiCAD_Sym:RES -> SAMPI:RES
- R18: symbol Triet_KiCAD_Sym:RES -> SAMPI:RES
- R22: value 5.1K, 1% -> 5.1K; symbol Triet_KiCAD_Sym:RES -> SAMPI:RES
Connections:
- net TXD_MCU is gone; now on net MCU_TXD: U4.44 (CK/TX/RC6)
- net +3.3V: now also R21.2, R23.2
- net +VDDTG: now also R22.2, R19.2, R20.2, R27.1, R35.1; no longer R22.1
- net GND: now also C15.2, C17.2, C14.2, C21.1, C22.2, R12.1, R13.1, R14.1, R15.1, R16.1, R17.1, R33.2, R9.1, U6.3 (GND); no longer C15.1, C17.1
- net GPIO: now also U4.15 (RB5); no longer U4.27 (RE2/~{CS}/AN7)
- net RD0: now also U4.5 (RD7/PSP7); no longer U4.38 (RD0/PSP0)
- net RD1: now also U4.4 (RD6/PSP6); no longer U4.39 (RD1/PSP1)
- net RD2: now also U4.3 (RD5/PSP5); no longer U4.40 (RD2/PSP2)
- net RD3: now also U4.2 (RD4/PSP4); no longer U4.41 (RD3/PSP3)
- net RD4: now also U4.41 (RD3/PSP3); no longer U4.2 (RD4/PSP4)
- net RD5: now also U4.40 (RD2/PSP2); no longer U4.3 (RD5/PSP5)
- net RD6: now also U4.39 (RD1/PSP1); no longer U4.4 (RD6/PSP6)
- net RD7: now also U4.38 (RD0/PSP0); no longer U4.5 (RD7/PSP7)
- net SCL: now also R22.1; no longer MD1.32 (D15/SCL), R22.2, U4.37 (SCK/SCL/RC3)
- net SCLK: now also U4.37 (SCK/SCL/RC3); no longer U4.15 (RB5)
- net SDA: now also R20.1; no longer MD1.31 (D14/SDA), U4.42 (SDI/SDA/RC4)
- net SDI: now also U4.42 (SDI/SDA/RC4); no longer U4.14 (RB4)
- net ~{CS}: now also U4.14 (RB4); no longer U4.26 (RE1/~{WR}/AN6)
- net ~{UBT}: now also C17.1; no longer C17.2
- net at J5.4 (SCL), Q6.2 (S): now also R21.1
- net at U10.3 (GND2), U4.30 (OSC1/CLKI): now also C15.1; no longer C15.2
- net at D8.K: now also R17.2
- net at D12.K: now also R13.2
- net at D10.K: now also R15.2
- net at J5.3 (SDA), Q7.2 (S): now also R23.1
- net at D11.K: now also R14.2
- net at D14.K: now also R9.2
- net at D9.K: now also R16.2
- net at D13.K: now also R12.2
- net PGC/UART_RX_IND renamed PGC_SDA
- net PGC_SDA: now also MD1.31 (D14/SDA), R27.2
- net PGD/UART_TX_SEL renamed PGD_SCL
- net PGD_SCL: now also MD1.32 (D15/SCL), R19.1
- net RXD: no longer names the net of MD1.15 (D0/RXD)
- net RXD: now also R32.1
- net RXD_MCU renamed MCU_TXD
- net MCU_TXD: now also R31.2, R32.2
- net TXD: no longer names the net of MD1.16 (D1/TXD)
- net TXD: now also R31.1
- new net: C21.2, R34.2, R35.2, U6.1 (VDD)
- new net LIGHT: U4.27 (RE2/~{CS}/AN7)
- new net TEMP: C14.1, C22.1, R33.1, R34.1, U4.26 (RE1/~{WR}/AN6), U6.2 (VOUT)
